Commit message: Rename package from puzzlebot_sim to puzzlebot_sim2 and update references in launch files, README, and configuration files.

File: MiniChallenge3/src/urdf/puzzlebot.urdf (robot description, URDF)
Before this commit: robot puzzlebot, 6 links, 5 joints
Links:
- link base_link: geometry collision box size=0.23 0.19 0.07; visual mesh filename=package://puzzlebot_sim2/meshes/Puzzlebot_Jetson_Lidar_Edit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
- link caster_holder_link: geometry collision box size=0.04 0.04 0.02; visual mesh filename=package://puzzlebot_sim2/meshes/Puzzlebot_Caster_Wheel.stl
- link wheel_left_link: geometry collision cylinder length=0.02 radius=0.033; visual mesh filename=package://puzzlebot_sim2/meshes/Puzzlebot_Wheel.stl
- link wheel_right_link: geometry collision cylinder length=0.02 radius=0.033; visual mesh filename=package://puzzlebot_sim2/meshes/Puzzlebot_Wheel.stl
