Commit message: Refactor Puzzlebot Simulation: Remove old nodes, add robot markers, and update URDF
- Deleted obsolete `puzzlebot_sim_node.py` and `trajectory_generator_node.py`.
- Introduced `robot_markers.py` for visualization of the Puzzlebot model in RViz.
- Updated URDF file to reflect new mesh paths and simplified link definitions.
- Adjusted `setup.py` to include new file structure and updated maintainer information.
- Removed old RViz configuration file and replaced it with a new structure.

File: MiniChallenge3/src/puzzlebot_sim/urdf/puzzlebot.urdf (robot description, URDF)
Before this commit: robot puzzlebot, 6 links, 5 joints
Links:
- removed link caster_holder_link
- removed link wheel_caster_link
- removed link wheel_left_link
- removed link wheel_right_link
- added link caster; visual mesh filename=package://puzzlebot_sim/meshes/Puzzlebot_Caster_Wheel.stl scale=1 1 1
- added link wheel_l; visual mesh filename=package://puzzlebot_sim/meshes/Puzzlebot_Wheel.stl scale=1 1 1
- added link wheel_r; visual mesh filename=package://puzzlebot_sim/meshes/Puzzlebot_Wheel.stl scale=1 1 1
- link base_link: mass 2.0 -> None; geometry visual mesh filename=package://puzzlebot_sim/meshes/Puzzlebot_Jetson_Lidar_Editi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 scale=1 1 1
Joints:
- removed joint base_joint
- removed joint caster_holder_joint
- removed joint wheel_caster_joint
- removed joint wheel_left_joint
- removed joint wheel_right_joint
- added joint base_link_joint: type fixed, parent base_footprint, child base_link, origin xyz=0 0 0.05 rpy=0 0 0
- added joint caster_joint: type fixed, parent base_link, child caster, origin xyz=-0.095 0 -0.04 rpy=0 0 0
- added joint wheel_l_joint: type continuous, parent base_link, child wheel_l, origin xyz=0.052 0.095 -0.0025 rpy=0 0 0, axis 0 1 0
- added joint wheel_r_joint: type continuous, parent base_link, child wheel_r, origin xyz=0.052 -0.095 -0.0025 rpy=0 0 0, axis 0 1 0

Commit message: Add Bug0 architecture documentation, launch file, and implement Bug0 control logic for navigation and obstacle avoidance

File: MiniChallenge3/src/puzzlebot_sim/urdf/puzzlebot.urdf (robot description, URDF)
Before this commit: robot puzzlebot, 5 links, 4 joints
Links:
- link base_link: geometry visual box size=0.2 0.15 0.05
